Commit message: created urdf rig for car (without ackermann steering)

File: ros/gra_navigation/description/robot_core.xacro (robot description, xacro)
@@ -12,13 +12,11 @@
         <origin xyz="0 0 0"/>
     </joint> launch-prefix="bash -c 'sleep 5; $0 $@'"
-    <!-- chassis description goes here. It describes the chassis of the bot which is a 54cm x 54cm x 150cm box -->
+    <!-- chassis description goes here. Needs to be updated when accurate dimension of the car is known-->
     <link name="chassis">
         <visual>
-            <!-- by default, the origin is centred around the link origin, so offset it by half the height -->
-            <!-- <origin xyz="0 0 0.75" rpy="0 0 0"/> -->
-            <geometry>
-                <!-- <box size="0.54 0.54 1.5"/> -->
-                <mesh filename="package://gra_base/meshes/frame_ultra_low_poly.stl" scale="0.001 0.001 0.001"/>
-                <!-- <mesh filename="model://frame_ultra_low_poly.stl"/> -->
+            <origin xyz="0 0 0.3" rpy="0 0 0"/>
+            <geometry>
+                <box size="2.5 0.75 0.5"/>
+                <!-- <mesh filename="package://gra_base/meshes/frame_ultra_low_poly.stl" scale="0.001 0.001 0.001"/> -->
             </geometry>
             <material name="white"/>
@@ -26,17 +24,17 @@
         <!-- physics model -->
         <collision>
-            <origin xyz="0 0 0.77" rpy="0 0 0"/>
-            <geometry>
-                <cylinder length="1.54" radius="0.25"/>
-            </geometry>
-        </collision>
-        <xacro:inertial_cylinder mass="20" length="1.54" radius="0.25">
-            <origin xyz="0 0 0.77" rpy="0 0 0"/>
-        </xacro:inertial_cylinder>
+            <origin xyz="0 0 0.3" rpy="0 0 0"/>
+            <geometry>
+                <box size="2.5 0.75 0.5"/>
+            </geometry>
+        </collision>
+        <xacro:inertial_box mass="300" x="2.5" y="0.75" z="0.5">
+            <origin xyz="0 0 0.3" rpy="0 0 0"/>
+        </xacro:inertial_box>
     </link>
     <joint name="laser_joint" type="fixed">
         <parent link="chassis"/>
         <child link="laser"/>
-        <origin xyz="0 0 0.07" rpy="0 0 0"/>
+        <origin xyz="1 0 0.575" rpy="0 0 0"/>
     </joint>
     <link name="laser">
@@ -57,5 +55,5 @@
         <parent link="base_link"/>
         <child link="wheel_1"/>
-        <origin xyz="0.2 0 0" rpy="0 -${pi/2} 0"/>
+        <origin xyz="1.25 0.5 0.2" rpy="${pi/2} 0 0"/>
         <axis xyz="0 0 1"/>
     </joint>
@@ -63,14 +61,14 @@
         <visual>
             <geometry>
-                <cylinder length="0.038" radius="0.05" />
-            </geometry>
-            <material name="black"/>
-        </visual>
-        <collision>
-            <geometry>
-                <cylinder length="0.038" radius="0.05" />
-            </geometry>
-        </collision>
-        <xacro:inertial_cylinder mass="0.2" length="0.038" radius="0.05">
+                <cylinder length="0.25" radius="0.20" />
+            </geometry>
+            <material name="black"/>
+        </visual>
+        <collision>
+            <geometry>
+                <cylinder length="0.25" radius="0.20" />
+            </geometry>
+        </collision>
+        <xacro:inertial_cylinder mass="5" length="0.25" radius="0.20">
             <origin xyz="0 0 0" rpy="0 0 0"/>
         </xacro:inertial_cylinder>
@@ -89,5 +87,5 @@
         <parent link="base_link"/>
         <child link="wheel_2"/>
-        <origin xyz="-0.1 -0.1732050808 0" rpy="0 ${pi/2} ${pi/3}"/>
+        <origin xyz="1.25 -0.5 0.2" rpy="-${pi/2} 0 0"/>
         <axis xyz="0 0 1"/>
     </joint>
@@ -95,14 +93,14 @@
         <visual>
             <geometry>
-                <cylinder length="0.038" radius="0.05" />
-            </geometry>
-            <material name="black"/>
-        </visual>
-        <collision>
-            <geometry>
-                <cylinder length="0.038" radius="0.05" />
-            </geometry>
-        </collision>
-        <xacro:inertial_cylinder mass="0.2" length="0.038" radius="0.05">
+                <cylinder length="0.25" radius="0.20" />
+            </geometry>
+            <material name="black"/>
+        </visual>
+        <collision>
+            <geometry>
+                <cylinder length="0.25" radius="0.20" />
+            </geometry>
+        </collision>
+        <xacro:inertial_cylinder mass="5" length="0.25" radius="0.20">
             <origin xyz="0 0 0" rpy="0 0 0"/>
         </xacro:inertial_cylinder>
@@ -121,5 +119,5 @@
         <parent link="base_link"/>
         <child link="wheel_3"/>
-        <origin xyz="-0.1 0.1732050808 0" rpy="0 ${pi/2} -${pi/3}"/>
+        <origin xyz="-1.25 -0.5 0.2" rpy="-${pi/2} 0 0"/>
         <axis xyz="0 0 1"/>
     </joint>
@@ -127,18 +125,50 @@
         <visual>
             <geometry>
-                <cylinder length="0.038" radius="0.05" />
-            </geometry>
-            <material name="black"/>
-        </visual>
-        <collision>
-            <geometry>
-                <cylinder length="0.038" radius="0.05" />
-            </geometry>
-        </collision>
-        <xacro:inertial_cylinder mass="0.2" length="0.038" radius="0.05">
+                <cylinder length="0.25" radius="0.20" />
+            </geometry>
+            <material name="black"/>
+        </visual>
+        <collision>
+            <geometry>
+                <cylinder length="0.25" radius="0.20" />
+            </geometry>
+        </collision>
+        <xacro:inertial_cylinder mass="5" length="0.25" radius="0.20">
             <origin xyz="0 0 0" rpy="0 0 0"/>
         </xacro:inertial_cylinder>
     </link>
     <gazebo reference="wheel_3">
+        <material>Gazebo/Black</material>
+        <mu1 value="0.2"/>
+        <mu2 value="1.5"/>
+        <kp value="10000000.0" />
+        <kd value="10000.0" />
+        <fdir1 value="0 0 1"/>
+        <maxContacts value= "1"/>
+    </gazebo>
+        <!-- WHEEL 4 -->
+    <joint name="wheel_4_joint" type="continuous">
+        <parent link="base_link"/>
+        <child link="wheel_4"/>
+        <origin xyz="-1.25 0.5 0.2" rpy="${pi/2} 0 0"/>
+        <axis xyz="0 0 1"/>
+    </joint>
+    <link name="wheel_4">
+        <visual>
+            <geometry>
+                <cylinder length="0.25" radius="0.20" />
+            </geometry>
+            <material name="black"/>
+        </visual>
+        <collision>
+            <geometry>
+                <cylinder length="0.25" radius="0.20" />
+            </geometry>
+        </collision>
+        <xacro:inertial_cylinder mass="5" length="0.25" radius="0.20">
+            <origin xyz="0 0 0" rpy="0 0 0"/>
+        </xacro:inertial_cylinder>
+    </link>
+    <gazebo reference="wheel_4">
         <material>Gazebo/Black</material>
         <mu1 value="0.2"/>

Commit message: added steering joint
although this version of steering joints will probably work, it is not accurate.(it steers both front wheels relative to centre point)

File: ros/gra_navigation/description/robot_core.xacro (robot description, xacro)
@@ -179,4 +179,37 @@
         <maxContacts value= "1"/>
     </gazebo>
+    <!-- Common Steering Link -->
+    <link name="front_steering_link">
+        <visual>
+            <geometry>
+                <box size="0.1 1.0 0.1"/>
+            </geometry>
+            <material name="white"/>
+        </visual>
+        <collision>
+            <geometry>
+                <box size="0.1 1.0 0.1"/>
+            </geometry>
+        </collision>
+    </link>
+    <!-- Joint connecting base_link to common steering link -->
+    <joint name="front_steering_joint" type="revolute">
+        <parent link="base_link"/>
+        <child link="front_steering_link"/>
+        <origin xyz="1.25 0 0.2" rpy="0 0 0"/>
+        <axis xyz="0 0 1"/>
+        <limit lower="-0.5236" upper="0.5236" effort="100" velocity="1"/> <!-- -30 to 30 degrees in radians -->
+    </joint>
+    <!-- Fixed joints connecting front wheels to common steering link -->
+    <joint name="wheel_1_to_steering_joint" type="fixed">
+        <parent link="front_steering_link"/>
+        <child link="wheel_1"/>
+        <origin xyz="0 0.5 0" rpy="${pi/2} 0 0"/>
+    </joint>
+    <joint name="wheel_2_to_steering_joint" type="fixed">
+        <parent link="front_steering_link"/>
+        <child link="wheel_2"/>
+        <origin xyz="0 -0.5 0" rpy="-${pi/2} 0 0"/>
+    </joint>
     <!-- Transmissions -->
     <transmission name="tran1">

Commit message: updated with the correct joints configuration
visual does not reflect steering

File: ros/gra_navigation/description/robot_core.xacro (robot description, xacro)
@@ -179,9 +179,24 @@
         <maxContacts value= "1"/>
     </gazebo>
-    <!-- Common Steering Link -->
-    <link name="front_steering_link">
-        <visual>
-            <geometry>
-                <box size="0.1 1.0 0.1"/>
+        <!-- WHEEL 1 Steering Joint -->
+    <joint name="wheel_1_steering_joint" type="revolute">
+        <parent link="base_link"/>
+        <child link="wheel_1_steering_link"/>
+        <origin xyz="1.25 0.5 0.2" rpy="0 0 0"/>
+        <axis xyz="0 0 1"/>
+        <limit lower="-0.5236" upper="0.5236" effort="100" velocity="1"/> <!-- -30 to 30 degrees in radians -->
+    </joint>
+    <!-- WHEEL 1 Driving Joint -->
+    <joint name="wheel_1_driving_joint" type="fixed">
+        <parent link="wheel_1_steering_link"/>
+        <child link="wheel_1"/>
+        <origin xyz="0 0 0" rpy="${pi/2} 0 0"/>
+        <axis xyz="0 1 0"/>
+    </joint>
+    <!-- Add a steering link for wheel_1 -->
+    <link name="wheel_1_steering_link">
+        <visual>
+            <geometry>
+                <box size="0.1 0.1 0.1"/>
             </geometry>
             <material name="white"/>
@@ -189,27 +204,37 @@
         <collision>
             <geometry>
-                <box size="0.1 1.0 0.1"/>
-            </geometry>
-        </collision>
-    </link>
-    <!-- Joint connecting base_link to common steering link -->
-    <joint name="front_steering_joint" type="revolute">
-        <parent link="base_link"/>
-        <child link="front_steering_link"/>
-        <origin xyz="1.25 0 0.2" rpy="0 0 0"/>
+                <box size="0.1 0.1 0.1"/>
+            </geometry>
+        </collision>
+    </link>
+    <!-- WHEEL 2 Steering Joint -->
+    <joint name="wheel_2_steering_joint" type="revolute">
+        <parent link="base_link"/>
+        <child link="wheel_2_steering_link"/>
+        <origin xyz="1.25 -0.5 0.2" rpy="0 0 0"/>
         <axis xyz="0 0 1"/>
         <limit lower="-0.5236" upper="0.5236" effort="100" velocity="1"/> <!-- -30 to 30 degrees in radians -->
     </joint>
-    <!-- Fixed joints connecting front wheels to common steering link -->
-    <joint name="wheel_1_to_steering_joint" type="fixed">
-        <parent link="front_steering_link"/>
-        <child link="wheel_1"/>
-        <origin xyz="0 0.5 0" rpy="${pi/2} 0 0"/>
-    </joint>
-    <joint name="wheel_2_to_steering_joint" type="fixed">
-        <parent link="front_steering_link"/>
+    <!-- WHEEL 2 Driving Joint -->
+    <joint name="wheel_2_driving_joint" type="fixed">
+        <parent link="wheel_2_steering_link"/>
         <child link="wheel_2"/>
-        <origin xyz="0 -0.5 0" rpy="-${pi/2} 0 0"/>
-    </joint>
+        <origin xyz="0 0 0" rpy="-${pi/2} 0 0"/>
+        <axis xyz="0 1 0"/>
+    </joint>
+    <!-- Add a steering link for wheel_2 -->
+    <link name="wheel_2_steering_link">
+        <visual>
+            <geometry>
+                <box size="0.1 0.1 0.1"/>
+            </geometry>
+            <material name="white"/>
+        </visual>
+        <collision>
+            <geometry>
+                <box size="0.1 0.1 0.1"/>
+            </geometry>
+        </collision>
+    </link>
     <!-- Transmissions -->
     <transmission name="tran1">
@@ -250,4 +275,24 @@
         <actuator name="motor_4">
             <hardwareInterface>VelocityJointInterface</hardwareInterface>
+            <mechanicalReduction>1</mechanicalReduction>
+        </actuator>
+    </transmission>
+    <transmission name="steering_tran1">
+        <type>transmission_interface/SimpleTransmission</type>
+        <joint name="wheel_1_steering_joint">
+            <hardwareInterface>hardware_interface/PositionJointInterface</hardwareInterface>
+        </joint>
+        <actuator name="steering_motor_1">
+            <hardwareInterface>PositionJointInterface</hardwareInterface>
+            <mechanicalReduction>1</mechanicalReduction>
+        </actuator>
+    </transmission>
+    <transmission name="steering_tran2">
+        <type>transmission_interface/SimpleTransmission</type>
+        <joint name="wheel_2_steering_joint">
+            <hardwareInterface>hardware_interface/PositionJointInterface</hardwareInterface>
+        </joint>
+        <actuator name="steering_motor_2">
+            <hardwareInterface>PositionJointInterface</hardwareInterface>
             <mechanicalReduction>1</mechanicalReduction>
         </actuator>

Commit message: Revert "updated with the correct joints configuration"
This reverts commit 55d26e9625886aaeee200fe1fd37aa4e048e7f90.

File: ros/gra_navigation/description/robot_core.xacro (robot description, xacro)
@@ -179,62 +179,37 @@
         <maxContacts value= "1"/>
     </gazebo>
-        <!-- WHEEL 1 Steering Joint -->
-    <joint name="wheel_1_steering_joint" type="revolute">
-        <parent link="base_link"/>
-        <child link="wheel_1_steering_link"/>
-        <origin xyz="1.25 0.5 0.2" rpy="0 0 0"/>
+    <!-- Common Steering Link -->
+    <link name="front_steering_link">
+        <visual>
+            <geometry>
+                <box size="0.1 1.0 0.1"/>
+            </geometry>
+            <material name="white"/>
+        </visual>
+        <collision>
+            <geometry>
+                <box size="0.1 1.0 0.1"/>
+            </geometry>
+        </collision>
+    </link>
+    <!-- Joint connecting base_link to common steering link -->
+    <joint name="front_steering_joint" type="revolute">
+        <parent link="base_link"/>
+        <child link="front_steering_link"/>
+        <origin xyz="1.25 0 0.2" rpy="0 0 0"/>
         <axis xyz="0 0 1"/>
         <limit lower="-0.5236" upper="0.5236" effort="100" velocity="1"/> <!-- -30 to 30 degrees in radians -->
     </joint>
-    <!-- WHEEL 1 Driving Joint -->
-    <joint name="wheel_1_driving_joint" type="fixed">
-        <parent link="wheel_1_steering_link"/>
+    <!-- Fixed joints connecting front wheels to common steering link -->
+    <joint name="wheel_1_to_steering_joint" type="fixed">
+        <parent link="front_steering_link"/>
         <child link="wheel_1"/>
-        <origin xyz="0 0 0" rpy="${pi/2} 0 0"/>
-        <axis xyz="0 1 0"/>
-    </joint>
-    <!-- Add a steering link for wheel_1 -->
-    <link name="wheel_1_steering_link">
-        <visual>
-            <geometry>
-                <box size="0.1 0.1 0.1"/>
-            </geometry>
-            <material name="white"/>
-        </visual>
-        <collision>
-            <geometry>
-                <box size="0.1 0.1 0.1"/>
-            </geometry>
-        </collision>
-    </link>
-    <!-- WHEEL 2 Steering Joint -->
-    <joint name="wheel_2_steering_joint" type="revolute">
-        <parent link="base_link"/>
-        <child link="wheel_2_steering_link"/>
-        <origin xyz="1.25 -0.5 0.2" rpy="0 0 0"/>
-        <axis xyz="0 0 1"/>
-        <limit lower="-0.5236" upper="0.5236" effort="100" velocity="1"/> <!-- -30 to 30 degrees in radians -->
-    </joint>
-    <!-- WHEEL 2 Driving Joint -->
-    <joint name="wheel_2_driving_joint" type="fixed">
-        <parent link="wheel_2_steering_link"/>
+        <origin xyz="0 0.5 0" rpy="${pi/2} 0 0"/>
+    </joint>
+    <joint name="wheel_2_to_steering_joint" type="fixed">
+        <parent link="front_steering_link"/>
         <child link="wheel_2"/>
-        <origin xyz="0 0 0" rpy="-${pi/2} 0 0"/>
-        <axis xyz="0 1 0"/>
-    </joint>
-    <!-- Add a steering link for wheel_2 -->
-    <link name="wheel_2_steering_link">
-        <visual>
-            <geometry>
-                <box size="0.1 0.1 0.1"/>
-            </geometry>
-            <material name="white"/>
-        </visual>
-        <collision>
-            <geometry>
-                <box size="0.1 0.1 0.1"/>
-            </geometry>
-        </collision>
-    </link>
+        <origin xyz="0 -0.5 0" rpy="-${pi/2} 0 0"/>
+    </joint>
     <!-- Transmissions -->
     <transmission name="tran1">
@@ -275,24 +250,4 @@
         <actuator name="motor_4">
             <hardwareInterface>VelocityJointInterface</hardwareInterface>
-            <mechanicalReduction>1</mechanicalReduction>
-        </actuator>
-    </transmission>
-    <transmission name="steering_tran1">
-        <type>transmission_interface/SimpleTransmission</type>
-        <joint name="wheel_1_steering_joint">
-            <hardwareInterface>hardware_interface/PositionJointInterface</hardwareInterface>
-        </joint>
-        <actuator name="steering_motor_1">
-            <hardwareInterface>PositionJointInterface</hardwareInterface>
-            <mechanicalReduction>1</mechanicalReduction>
-        </actuator>
-    </transmission>
-    <transmission name="steering_tran2">
-        <type>transmission_interface/SimpleTransmission</type>
-        <joint name="wheel_2_steering_joint">
-            <hardwareInterface>hardware_interface/PositionJointInterface</hardwareInterface>
-        </joint>
-        <actuator name="steering_motor_2">
-            <hardwareInterface>PositionJointInterface</hardwareInterface>
             <mechanicalReduction>1</mechanicalReduction>
         </actuator>

Commit message: imported chassis mesh

File: ros/gra_navigation/description/robot_core.xacro (robot description, xacro)
@@ -17,6 +17,6 @@
             <origin xyz="0 0 0.3" rpy="0 0 0"/>
             <geometry>
-                <box size="2.5 0.75 0.5"/>
-                <!-- <mesh filename="package://gra_base/meshes/frame_ultra_low_poly.stl" scale="0.001 0.001 0.001"/> -->
+                <!-- <box size="2.5 0.75 0.5"/> -->
+                <mesh filename="package://gra_base/meshes/ads-dv.stl"/>
             </geometry>
             <material name="white"/>

Commit message: repositioned LIDAR

File: ros/gra_navigation/description/robot_core.xacro (robot description, xacro)
@@ -36,5 +36,5 @@
         <parent link="chassis"/>
         <child link="laser"/>
-        <origin xyz="1 0 0.575" rpy="0 0 0"/>
+        <origin xyz="0.1 0 0.75" rpy="0 0 0"/>
     </joint>
     <link name="laser">
