Commit message: removed battery

File: ros/ackermann_vehicle_description/urdf/em_3905_hokuyo.urdf.xacro (robot description, xacro)
@@ -38,16 +38,4 @@
   <xacro:property name="chassis_height" value="0.01"/>
   <xacro:property name="chassis_mass" value="2.788"/>
-  <!-- battery_dist is the distance between the inner edges of the
-       batteries. battery_comp_depth is the battery compartment depth.
-       battery_length is measured along the x axis, battery_width
-       along the y axis, and battery_height along the z axis. -->
-  <xacro:property name="battery_x_offset" value="0.055"/>
-  <xacro:property name="battery_dist" value="0.065"/>
-  <xacro:property name="battery_comp_depth" value="0.02"/>
-  <xacro:property name="battery_comp_angle" value="0.34906585"/>
-  <xacro:property name="battery_length" value="0.16"/>
-  <xacro:property name="battery_width" value="0.047"/>
-  <xacro:property name="battery_height" value="0.024"/>
-  <xacro:property name="battery_mass" value="0.5025"/>
   <!-- hub_dia and tire_dia are the diameters of the hub and tire,
        respectively. hex_hub_depth is the distance that the hex hub is
@@ -94,7 +82,4 @@
   <xacro:property name="servo_stall_torque" value="0.5649"/>
   <xacro:property name="servo_no_load_speed" value="4.553"/>
-  <material name="battery_mat">
-    <color rgba="0 0 1 1"/>
-  </material>
   <material name="chassis_mat">
     <color rgba="0.5 0.5 0.5 1"/>
@@ -141,46 +126,4 @@
                     outer_rad * outer_rad) / 2}"/>
     </inertial>
-  </xacro:macro>
-  <!-- Battery -->
-  <xacro:macro name="battery" params="prefix reflect">
-    <joint name="chassis_to_${prefix}_battery" type="fixed">
-      <parent link="chassis"/>
-      <child link="${prefix}_battery_offset"/>
-      <origin xyz="${battery_x_offset - battery_length / 2}
-                   ${reflect * battery_dist / 2}
-                   0"
-              rpy="${reflect * battery_comp_angle} 0 0"/>
-    </joint>
-    <link name="${prefix}_battery_offset">
-      <xacro:null_inertial/>
-    </link>
-    <joint name="offset_to_${prefix}_battery" type="fixed">
-      <parent link="${prefix}_battery_offset"/>
-      <child link="${prefix}_battery"/>
-      <origin xyz="0
-                   ${reflect * battery_width / 2}
-                   ${(battery_height / 2) - battery_comp_depth}"/>
-    </joint>
-    <link name="${prefix}_battery">
-      <visual>
-        <geometry>
-          <box size="${battery_length} ${battery_width} ${battery_height}"/>
-        </geometry>
-        <material name="battery_mat"/>
-      </visual>
-      <collision>
-        <geometry>
-          <box size="${battery_length} ${battery_width} ${battery_height}"/>
-        </geometry>
-      </collision>
-      <xacro:solid_cuboid_inertial
-         width="${battery_length}" depth="${battery_width}"
-         height="${battery_height}" mass="${battery_mass}">
-        <origin/>
-      </xacro:solid_cuboid_inertial>
-    </link>
-    <gazebo reference="${prefix}_battery">
-      <material>Gazebo/Blue</material>
-    </gazebo>
   </xacro:macro>
   <!-- Shock absorber -->
@@ -345,7 +288,4 @@
     <child link="chassis"/>
   </joint>
-  <!-- Batteries -->
-  <xacro:battery prefix="left" reflect="1"/>
-  <xacro:battery prefix="right" reflect="-1"/>
   <!-- Wheels -->
   <xacro:front_wheel lr_prefix="left" fr_prefix="front"

Commit message: changed chassis colour

File: ros/ackermann_vehicle_description/urdf/em_3905_hokuyo.urdf.xacro (robot description, xacro)
@@ -83,5 +83,5 @@
   <xacro:property name="servo_no_load_speed" value="4.553"/>
   <material name="chassis_mat">
-    <color rgba="0.5 0.5 0.5 1"/>
+    <color rgba="0.0 0.2 0.13 1"/>
   </material>
   <material name="tire_mat">
@@ -265,5 +265,6 @@
       <origin xyz="0 0 ${-chassis_height / 2}"/>
       <geometry>
-        <box size="${chassis_length} ${chassis_width} ${chassis_height}"/>
+        <!-- <box size="${chassis_length} ${chassis_width} ${chassis_height}"/> -->
+        <mesh filename="package://ackermann_vehicle_description/meshes/ads-dv.stl" scale="0.25 0.25 0.25"/>
       </geometry>
       <material name="chassis_mat"/>
@@ -282,5 +283,5 @@
   </link>
   <gazebo reference="chassis">
-    <material>Gazebo/Grey</material>
+    <material>Gazebo/Grass</material>
   </gazebo>
   <joint name="base_link_to_chassis" type="fixed">

Commit message: depth camera now operational in gazebo

File: ros/ackermann_vehicle_description/urdf/em_3905_hokuyo.urdf.xacro (robot description, xacro)
@@ -338,3 +338,71 @@
   </xacro:macro>
   <xacro:hokuyo_laser/>
+  <!-- Depth Camera -->
+  <joint name="camera_joint" type="fixed">
+    <parent link="base_link" />
+    <child link="camera_link" />
+    <origin xyz="0.065 0 0.075" rpy="0 0 0" />
+  </joint>
+  <link name="camera_link">
+    <visual>
+      <geometry>
+        <box size="0.02 0.1 0.03"/>
+      </geometry>
+    </visual>
+    <!-- <inertial>
+      <mass value="0.001"/>
+      <origin xyz="0 0 0"/>
+      <inertia ixx="0.0001" ixy="0.0" ixz="0.0" iyy="0.0001" iyz="0.0" izz="0.0001"/>
+    </inertial> -->
+  </link>
+  <joint name="camera_optical_joint" type="fixed">
+    <parent link="camera_link"/>
+    <child link="camera_link_optical"/>
+    <origin xyz="0 0 0" rpy="${-pi/2} 0 ${-pi/2}" />
+  </joint>
+  <link name="camera_link_optical"></link>
+  <gazebo reference="camera_link">
+    <material>Gazebo/Blue</material>
+    <sensor name="camera" type="depth">
+      <pose>0 0 0 0 0 0</pose>
+      <visualize>true</visualize>
+      <update_rate>30</update_rate>
+      <camera>
+        <horizontal_fov>1.204</horizontal_fov>
+        <image>
+          <width>640</width>
+          <height>480</height>
+          <format>B8G8R8</format>
+        </image>
+        <clip>
+          <near>0.05</near>
+          <far>8.0</far>
+        </clip>
+      </camera>
+      <plugin name="camera_controller" filename="libgazebo_ros_openni_kinect.so">
+        <frameName>camera_link_optical</frameName>
+        <baseline>0.2</baseline>
+        <alwaysOn>true</alwaysOn>
+        <updateRate>30.0</updateRate>
+        <!-- <cameraName>ackermann_vehicle_ir</cameraName> -->
+        <imageTopicName>/ackermann_vehicle/color/image_raw</imageTopicName>
+        <cameraInfoTopicName>/ackermann_vehicle/color/camera_info</cameraInfoTopicName>
+        <depthImageTopicName>/ackermann_vehicle/depth/image_raw</depthImageTopicName>
+        <depthImageInfoTopicName>/ackermann_vehicle/depth/camera_info</depthImageInfoTopicName>
+        <pointCloudTopicName>/ackermann_vehicle/depth/points</pointCloudTopicName>
+        <pointCloudCutoff>0.5</pointCloudCutoff>
+        <pointCloudCutoffMax>3.0</pointCloudCutoffMax>
+        <distortionK1>0.00000001</distortionK1>
+        <distortionK2>0.00000001</distortionK2>
+        <distortionK3>0.00000001</distortionK3>
+        <distortionT1>0.00000001</distortionT1>
+        <distortionT2>0.00000001</distortionT2>
+        <CxPrime>0</CxPrime>
+        <Cx>0</Cx>
+        <Cy>0</Cy>
+        <focalLength>0</focalLength>
+        <hackBaseline>0</hackBaseline>
+      </plugin>
+    </sensor>
+  </gazebo>
 </robot>

Commit message: Update em_3905_hokuyo.urdf.xacro

File: ros/ackermann_vehicle_description/urdf/em_3905_hokuyo.urdf.xacro (robot description, xacro)
@@ -276,5 +276,5 @@
                     lr_reflect="-1" fr_reflect="-1"/>
   <!-- LiDAR -->
-  <link name="hokuyo_link">
+  <link name="laser">
     <visual>
       <geometry>
@@ -292,5 +292,5 @@
     <origin xyz="-0.065 0 0.075" rpy="0 0 0" />
     <parent link="base_link" />
-    <child link="hokuyo_link" />
+    <child link="laser" />
   </joint>
   <gazebo>
@@ -332,5 +332,5 @@
         <plugin name="gazebo_ros_head_hokuyo_controller" filename="libgazebo_ros_laser.so">
           <topicName>/ackermann_vehicle/scan</topicName>
-          <frameName>hokuyo_link</frameName>
+          <frameName>laser</frameName>
         </plugin>
       </sensor>

Commit message: rosbag track run & lidar re orientation
2 track runs; lidar rotated 180 deg in z axis

File: ros/ackermann_vehicle_description/urdf/em_3905_hokuyo.urdf.xacro (robot description, xacro)
@@ -290,5 +290,5 @@
   </link>
   <joint name="laser_joint" type="fixed">
-    <origin xyz="-0.065 0 0.075" rpy="0 0 0" />
+    <origin xyz="-0.065 0 0.075" rpy="0 0 ${pi}" />
     <parent link="base_link" />
     <child link="laser" />

Commit message: Added 3D lidar to urdf

File: ros/ackermann_vehicle_description/urdf/em_3905_hokuyo.urdf.xacro (robot description, xacro)
@@ -275,5 +275,5 @@
   <xacro:rear_wheel lr_prefix="right" fr_prefix="rear"
                     lr_reflect="-1" fr_reflect="-1"/>
-  <!-- LiDAR -->
+  <!-- 2D LiDAR -->
   <link name="laser">
     <visual>
@@ -338,4 +338,26 @@
   </xacro:macro>
   <xacro:hokuyo_laser/>
+  <!-- 3D LiDAR (VLP-16) Frame -->
+  <link name="velodyne">
+    <visual>
+      <origin xyz="0 0 0.09" rpy="0 0 0"/> <!-- Adjust the z-offset as needed -->
+      <geometry>
+        <cylinder radius="0.05" length="0.07"/>
+      </geometry>
+      <material name="lidar_mat">
+        <color rgba="0.5 0.5 0.5 1"/>
+      </material>
+    </visual>
+    <inertial>
+      <mass value="0.1"/> <!-- Adjust the mass as needed -->
+      <origin xyz="0 0 0"/>
+      <inertia ixx="0.0005" ixy="0" ixz="0" iyy="0.0005" iyz="0" izz="0.0005"/>
+    </inertial>
+  </link>
+  <joint name="velodyne_joint" type="fixed">
+    <parent link="base_link"/> <!-- Ensure this is the correct parent link -->
+    <child link="velodyne"/>
+    <origin xyz="0 0 0.09" rpy="0 0 0"/> <!-- Adjust xyz for positioning, rpy for orientation -->
+  </joint>
   <!-- Depth Camera -->
   <joint name="camera_joint" type="fixed">

Commit message: Fixed small scale urdf laser orientation

File: ros/ackermann_vehicle_description/urdf/em_3905_hokuyo.urdf.xacro (robot description, xacro)
@@ -289,5 +289,5 @@
   </link>
   <joint name="laser_joint" type="fixed">
-    <origin xyz="-0.065 0 0.075" rpy="0 0 ${pi}" />
+    <origin xyz="-0.065 0 0.075" rpy="0 0 0" />
     <parent link="base_link" />
     <child link="laser" />
@@ -304,5 +304,5 @@
         <pose>0 0 0 0 0 0</pose>
         <visualize>true</visualize>
-        <update_rate>40</update_rate>
+        <update_rate>100</update_rate>
         <ray>
           <scan>
@@ -310,10 +310,10 @@
               <samples>720</samples>
               <resolution>1</resolution>
-              <min_angle>-1.570796</min_angle>
-              <max_angle>1.570796</max_angle>
+              <min_angle>-${M_PI}</min_angle>
+              <max_angle>${M_PI}</max_angle>
             </horizontal>
           </scan>
           <range>
-            <min>0.10</min>
+            <min>0.40</min>
             <max>80.0</max>
             <resolution>0.01</resolution>
