Commit message: Rewired all ads-dv sensors to attach to base_link instead of chassis

File: ros/ackermann_vehicle_description/urdf/ads_dv.urdf.xacro (robot description, xacro)
@@ -291,6 +291,6 @@
   </link>
   <joint name="laser_joint" type="fixed">
-    <origin xyz="0.3 0 0.27" rpy="0 0 ${pi}" />
-    <parent link="chassis" />
+    <origin xyz="0.3 0 ${chassis_height/2 + 0.27}" rpy="0 0 ${pi}" />
+    <parent link="base_link" />
     <child link="laser" />
   </joint>
@@ -298,6 +298,6 @@
     <plugin name="gazebo_ros_control" filename="libgazebo_ros_control.so"/>
   </gazebo>
-  <xacro:hokuyo_utm30lx_model name="hokuyo_laser" parent="chassis">
-    <origin xyz="0.3 0 0.27" rpy="0 0 0" />
+  <xacro:hokuyo_utm30lx_model name="hokuyo_laser" parent="base_link">
+    <origin xyz="0.3 0 ${chassis_height/2+0.27}" rpy="0 0 0" />
   </xacro:hokuyo_utm30lx_model>
   <xacro:macro name="hokuyo_laser">
@@ -357,7 +357,7 @@
   </link>
   <joint name="velodyne_joint" type="fixed">
-    <parent link="chassis"/> <!-- Ensure this is the correct parent link -->
+    <parent link="base_link"/> <!-- Ensure this is the correct parent link -->
     <child link="velodyne"/>
-    <origin xyz="0.4 0 0.27" rpy="0 0 0"/> <!-- Adjust xyz for positioning, rpy for orientation -->
+    <origin xyz="0.4 0 ${chassis_height/2 + 0.27}" rpy="0 0 0"/> <!-- Adjust xyz for positioning, rpy for orientation -->
   </joint>
   <gazebo reference="velodyne">
@@ -365,9 +365,9 @@
       <pose>0 0 0 0 0 0</pose>
       <visualize>false</visualize>
-      <update_rate>8</update_rate>
+      <update_rate>5</update_rate>
       <ray>
         <scan>
           <horizontal>
-            <samples>700</samples>
+            <samples>600</samples>
             <resolution>1</resolution>
             <min_angle>-${M_PI}</min_angle>
@@ -383,5 +383,5 @@
         <range>
           <min>2</min>
-          <max>26</max>
+          <max>81</max>
           <resolution>0.01</resolution>
         </range>
@@ -396,5 +396,5 @@
         <frameName>velodyne</frameName>
         <min_range>2</min_range>
-        <max_range>25.0</max_range>
+        <max_range>80.0</max_range>
         <!-- <gaussianNoise>0.008</gaussianNoise> -->
         <gaussianNoise>0</gaussianNoise>
@@ -404,8 +404,8 @@
   <!-- Depth Camera -->
   <joint name="camera_joint" type="fixed">
-    <parent link="chassis" />
+    <parent link="base_link" />
     <child link="camera_link" />
     <!-- <origin xyz="0.08 0 0.425" rpy="0 0 0" /> -->
-    <origin xyz="1.4 0 0.05" rpy="0 0 0" />
+    <origin xyz="1.4 0 ${chassis_height/2 + 0.05}" rpy="0 0 0" />
   </joint>
   <link name="camera_link">

Commit message: New odometry model working, but require tuning

File: ros/ackermann_vehicle_description/urdf/ads_dv.urdf.xacro (robot description, xacro)
@@ -242,5 +242,4 @@
       <origin xyz="-0.1 0 0"/>
       <geometry>
-        <!-- <box size="${chassis_length} ${chassis_width} ${chassis_height}"/> -->
         <mesh filename="package://ackermann_vehicle_description/meshes/ads-dv.stl" scale="1 1 1"/>
       </geometry>
@@ -342,5 +341,5 @@
   <link name="velodyne">
     <visual>
-      <origin xyz="0 0 0" rpy="0 0 0"/> <!-- Adjust the z-offset as needed -->
+      <origin xyz="0 0 0" rpy="0 0 0"/>
       <geometry>
         <cylinder radius="0.05" length="0.07"/>
@@ -351,5 +350,5 @@
     </visual>
     <inertial>
-      <mass value="0.1"/> <!-- Adjust the mass as needed -->
+      <mass value="0.1"/>
       <origin xyz="0 0 0"/>
       <inertia ixx="0.0005" ixy="0" ixz="0" iyy="0.0005" iyz="0" izz="0.0005"/>
@@ -357,7 +356,7 @@
   </link>
   <joint name="velodyne_joint" type="fixed">
-    <parent link="base_link"/> <!-- Ensure this is the correct parent link -->
+    <parent link="base_link"/>
     <child link="velodyne"/>
-    <origin xyz="0.4 0 ${chassis_height/2 + 0.27}" rpy="0 0 0"/> <!-- Adjust xyz for positioning, rpy for orientation -->
+    <origin xyz="0.4 0 ${chassis_height/2 + 0.27}" rpy="0 0 0"/>
   </joint>
   <gazebo reference="velodyne">

File: ros/ackermann_vehicle_description/urdf/em_3905_hokuyo.urdf.xacro (robot description, xacro)
@@ -242,5 +242,4 @@
       <origin xyz="0 0 ${-chassis_height / 2}"/>
       <geometry>
-        <!-- <box size="${chassis_length} ${chassis_width} ${chassis_height}"/> -->
         <mesh filename="package://ackermann_vehicle_description/meshes/ads-dv.stl" scale="0.25 0.25 0.25"/>
       </geometry>
@@ -341,5 +340,5 @@
   <link name="velodyne">
     <visual>
-      <origin xyz="0 0 0.09" rpy="0 0 0"/> <!-- Adjust the z-offset as needed -->
+      <origin xyz="0 0 0.09" rpy="0 0 0"/>
       <geometry>
         <cylinder radius="0.05" length="0.07"/>
@@ -350,5 +349,5 @@
     </visual>
     <inertial>
-      <mass value="0.1"/> <!-- Adjust the mass as needed -->
+      <mass value="0.1"/>
       <origin xyz="0 0 0"/>
       <inertia ixx="0.0005" ixy="0" ixz="0" iyy="0.0005" iyz="0" izz="0.0005"/>
@@ -356,7 +355,7 @@
   </link>
   <joint name="velodyne_joint" type="fixed">
-    <parent link="base_link"/> <!-- Ensure this is the correct parent link -->
+    <parent link="base_link"/>
     <child link="velodyne"/>
-    <origin xyz="0 0 0.09" rpy="0 0 0"/> <!-- Adjust xyz for positioning, rpy for orientation -->
+    <origin xyz="0 0 0.09" rpy="0 0 0"/>
   </joint>
   <gazebo reference="velodyne">

Commit message: Update ads_dv.urdf.xacro

File: ros/ackermann_vehicle_description/urdf/ads_dv.urdf.xacro (robot description, xacro)
@@ -358,5 +358,5 @@
     <parent link="base_link"/>
     <child link="velodyne"/>
-    <origin xyz="0.4 0 ${chassis_height/2 + 0.27}" rpy="0 0 0"/>
+    <origin xyz="0.667 0 ${chassis_height/2 + 0.27}" rpy="0 0 0"/>
   </joint>
   <gazebo reference="velodyne">
@@ -406,5 +406,5 @@
     <child link="camera_link" />
     <!-- <origin xyz="0.08 0 0.425" rpy="0 0 0" /> -->
-    <origin xyz="1.4 0 ${chassis_height/2 + 0.05}" rpy="0 0 0" />
+    <origin xyz="0.617 0 ${chassis_height/2 + 0.33}" rpy="0 0 0" />
   </joint>
   <link name="camera_link">

Commit message: Added real ads_dv launch file
no gazebo related nodes; uses 3D lidar graph slam; 3D lidar driver; depth camera driver

File: ros/ackermann_vehicle_description/urdf/ads_dv.urdf.xacro (robot description, xacro)
@@ -358,5 +358,5 @@
     <parent link="base_link"/>
     <child link="velodyne"/>
-    <origin xyz="0.667 0 ${chassis_height/2 + 0.27}" rpy="0 0 0"/>
+    <origin xyz="0.52 0 ${chassis_height/2 + 0.29246}" rpy="0 0 0"/>
   </joint>
   <gazebo reference="velodyne">
@@ -381,5 +381,5 @@
         </scan>
         <range>
-          <min>2</min>
+          <min>2.5</min>
           <max>81</max>
           <resolution>0.01</resolution>
@@ -394,5 +394,5 @@
         <topicName>/velodyne_points</topicName>
         <frameName>velodyne</frameName>
-        <min_range>2</min_range>
+        <min_range>2.5</min_range>
         <max_range>80.0</max_range>
         <!-- <gaussianNoise>0.008</gaussianNoise> -->
@@ -406,5 +406,5 @@
     <child link="camera_link" />
     <!-- <origin xyz="0.08 0 0.425" rpy="0 0 0" /> -->
-    <origin xyz="0.617 0 ${chassis_height/2 + 0.33}" rpy="0 0 0" />
+    <origin xyz="0.4865 0 ${chassis_height/2 + 0.364}" rpy="0 0 0" />
   </joint>
   <link name="camera_link">
